Commit message: Adding controlable joints and reasonable shape

File: 3dfiles/urdf/marcel.urdf (robot description, URDF)
Before this commit: robot marcel, 4 links, 3 joints
Links:
- removed link neck1
- removed link neck2
- added link neck; visual cylinder length=0.08 radius=0.025
- link base_link: geometry visual cylinder length=0.15 radius=0.1
- link face: geometry visual box size=0.035 0.12 0.18
Joints:
- removed joint neck1_to_neck2
- joint base_to_neck: axis (none) -> 0 0 1; child neck1 -> neck; limit (none) -> lower=${-2*pi/5} upper=${2*pi/5} effort=1000.0 velocity=5.0; origin xyz=0.0 0.0 1.60 rpy=0.0 -0.24 0.0 -> xyz=0.0 0.0 0.155 rpy=0.0 0.0 0.0; type fixed -> revolute
- joint neck_to_face: axis (none) -> 0 1 0; limit (none) -> lower=${-pi/2} upper=0.18 effort=1000.0 velocity=5.0; origin xyz=0.0 0.0 0.25 rpy=0.0 0.0 0.0 -> xyz=0.0 0.0 0.085 rpy=0.0 0.0 0.0; parent neck2 -> neck; type fixed -> revolute

Commit message: ROS/Gazebo/RViz updates: urdf with visual and fake physical info, useful ros launch commands stored

File: 3dfiles/urdf/marcel.urdf (robot description, URDF)
Before this commit: robot marcel, 3 links, 2 joints
Links:
- link base_link: mass None -> 1.0; geometry collision cylinder length=0.15 radius=0.1; visual cylinder length=0.15 radius=0.1
- link face: mass None -> 1.0; geometry collision box size=0.035 0.12 0.18; visual box size=0.035 0.12 0.18
- link neck: mass None -> 1.0; geometry collision cylinder length=0.08 radius=0.025; visual cylinder length=0.08 radius=0.025
